File: PCB/2026 DIT project.kicad_pcb (KiCad board)
At the start: 2 copper layers, 1 part

Commit message: PCB design process
Parts:
- added A1: SW_Push_Open_Dual, Button_Switch_THT:SW_PUSH_6mm, F.Cu at (31.8, 110.2)
- added B1: SW_Push_Open_Dual, Button_Switch_THT:SW_PUSH_6mm, F.Cu at (41.8, 110.2)
- added BZ1: Buzzer, Buzzer_Beeper:Buzzer_12x9.5RM7.6, F.Cu at (36.2, 95.5)
- added J1: Conn_01x07_Socket, Connector_PinHeader_2.54mm:PinHeader_1x07_P2.54mm_Vertical, F.Cu at (47.6, 118.5)
- added J2: Conn_01x04_Socket, Connector_PinSocket_2.54mm:PinSocket_1x04_P2.54mm_Vertical, F.Cu at (36.2, 84.5)
- added J3: Conn_01x05_Pin, Connector_PinHeader_2.54mm:PinHeader_1x05_P2.54mm_Vertical, F.Cu at (45.1, 122.5)
- added R1: 10k, Resistor_SMD:R_0805_2012Metric_Pad1.20x1.40mm_HandSolder, F.Cu at (38.0, 104.5)
- added R2: 10k, Resistor_SMD:R_0805_2012Metric_Pad1.20x1.40mm_HandSolder, F.Cu at (48.5, 104.0)
- U1: renamed from A1; value ~ -> ESP32-WROOM32U
- moved U1 1.64 mm to (25.5, 32.2)
Connections:
- U1 pad 0: unconnected-(A1-Pad0) -> /Buzzer
- U1 pad 16: unconnected-(A1-Pad16) -> /TXD
- U1 pad 17: unconnected-(A1-Pad17) -> /RXD
- U1 pad 2: unconnected-(A1-Pad2) -> /BTN_A
- U1 pad 21: unconnected-(A1-Pad21) -> /SDA
- U1 pad 22: unconnected-(A1-Pad22) -> /SCL
- U1 pad 3V3: unconnected-(A1-Pad3V3) -> +3V3
- U1 pad 4: unconnected-(A1-Pad4) -> /BTN_B
- U1 pad 5V: Net-(A1-Pad5V) -> +5V
- U1 pad CLK: Net-(A1-Pad5V) -> unconnected-(U1-PadCLK)
- U1 pad GND: unconnected-(A1-PadGND) -> GND
Other:
- board outline added: 34 x 99.5 mm
- board text added: "3.3V"
- board text added: "5V"
- board text added: "GND"
- board text added: "RXD"
- board text added: "TXD"

Commit message: PCB design complete
Parts:
- added BATT1: Screw_Terminal_01x02, TerminalBlock_Phoenix:TerminalBlock_Phoenix_MKDS-1,5-2-5.08_1x02_P5.08mm_Horizontal, F.Cu at (57.4, 117.0)
- added C1: 10u, Capacitor_SMD:C_0805_2012Metric_Pad1.18x1.45mm_HandSolder, F.Cu at (50.5, 118.5)
- added C2: 22u, Capacitor_SMD:C_0805_2012Metric_Pad1.18x1.45mm_HandSolder, F.Cu at (47.0, 126.8)
- added REF**: MountingHole_3.2mm_M3_DIN965_Pad, MountingHole:MountingHole_3.2mm_M3_DIN965_Pad, F.Cu at (21.5, 36.5)
- added REF**: MountingHole_3.2mm_M3_DIN965_Pad, MountingHole:MountingHole_3.2mm_M3_DIN965_Pad, F.Cu at (58.5, 36.5)
- added REF**: MountingHole_3.2mm_M3_DIN965_Pad, MountingHole:MountingHole_3.2mm_M3_DIN965_Pad, F.Cu at (21.5, 127.0)
- added REF**: MountingHole_3.2mm_M3_DIN965_Pad, MountingHole:MountingHole_3.2mm_M3_DIN965_Pad, F.Cu at (58.5, 127.0)
- added U2: AMS1117-5.0, Package_TO_SOT_SMD:SOT-89-3, F.Cu at (50.2, 123.2)
- moved A1 7.91 mm to (38.2, 114.8), turned to 180 degrees
- moved B1 7.91 mm to (48.2, 114.8), turned to 180 degrees
- moved R2 7.02 mm to (41.5, 104.5)
- moved R1 0.50 mm to (38.5, 104.5)
Connections:
- A1 pad 1: /BTN_A -> +3V3
- B1 pad 1: /BTN_B -> +3V3
Routing:
- net +5V: track 0.00 -> 117.6 mm, vias 0 -> 1
- net /TXD: track 0.00 -> 82.1 mm
- net /RXD: track 0.00 -> 81.4 mm, vias 0 -> 2
- net /BTN_A: track 0.00 -> 81.4 mm
- net +3V3: track 0.00 -> 77.7 mm
- net /BTN_B: track 0.00 -> 74.5 mm
- net /Buzzer: track 0.00 -> 59.2 mm
- net /SDA: track 0.00 -> 29.2 mm, vias 0 -> 2
- net /SCL: track 0.00 -> 20.5 mm, vias 0 -> 2
- net VCC: track 0.00 -> 10.1 mm
- added copper zone on B.Cu, net GND
- added copper zone on F.Cu, net GND
Other:
- board size 34 x 99.5 mm -> 46 x 99.5 mm
- board text added: "+"
- board text added: "-"
