File: PCB/2026 DIT project.kicad_sch (KiCad schematic)
At the start: 1 part

Commit message: PCB Design progress
Connections:
- net at A1.5V: no longer A1.CLK
Changed lines of the file:
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@@
 	(generator_version "9.0")
 	(paper "A4")
-	(wire
-		(pts
-			(xy 72.39 24.13) (xy 72.39 19.05)
-		)
-		(stroke
-			(width 0)
-			(type default)
-		)
-	)
-	(wire
-		(pts
-			(xy 76.2 24.13) (xy 72.39 24.13)
-		)
-		(stroke
-			(width 0)
-			(type default)
-		)
-	)
-	(wire
-		(pts
-			(xy 72.39 19.05) (xy 96.52 19.05)
-		)
-		(stroke
-			(width 0)
-			(type default)
-		)
-	)
-	(wire
-		(pts
-			(xy 96.52 19.05) (xy 96.52 24.13)
-		)
-		(stroke
-			(width 0)
-			(type default)
-		)
-	)
 	(image
 		(at 43.18 31.75)

Commit message: PCB design process
Parts:
- added A, B: SW_Push_Open_Dual, Button_Switch_THT:SW_PUSH_6mm, symbol Switch:SW_Push_Open_Dual
- added BZ1: Buzzer, Buzzer_Beeper:Buzzer_12x9.5RM7.6, symbol Device:Buzzer
- added J1: Conn_01x07_Socket, Connector_PinHeader_2.54mm:PinHeader_1x07_P2.54mm_Vertical, symbol Connector:Conn_01x07_Socket
- added J2: Conn_01x04_Socket, Connector_PinSocket_2.54mm:PinSocket_1x04_P2.54mm_Vertical, symbol Connector:Conn_01x04_Socket
- added J3: Conn_01x05_Pin, Connector_PinHeader_2.54mm:PinHeader_1x05_P2.54mm_Vertical, symbol Connector:Conn_01x05_Pin
- added R1, R2: 10k, Resistor_SMD:R_0805_2012Metric_Pad1.20x1.40mm_HandSolder, symbol Device:R
- U: renamed from A1; value ~ -> ESP32-WROOM32U
Connections:
- net Buzzer: now reaches U.0
- net Buzzer: now also BZ1.1 (+)
- net TXD: now reaches U.16
- net TXD: now also J1.4 (Pin_4), J3.2 (Pin_2)
- net RXD: now reaches U.17
- net RXD: now also J1.3 (Pin_3), J3.1 (Pin_1)
- net BTN_A: now reaches U.2
- net BTN_A: now also A.1, A.2, R1.1
- net SDA: now reaches U.21
- net SDA: now also J2.4 (Pin_4)
- net SCL: now reaches U.22
- net SCL: now also J2.3 (Pin_3)
- net +3V3: now reaches U.3V3
- net +3V3: now also A.3, A.4, B.3, B.4, J2.2 (Pin_2), J3.5 (Pin_5)
- net BTN_B: now reaches U.4
- net BTN_B: now also B.1, B.2, R2.1
- net +5V: now reaches U.5V
- net +5V: now also J1.6 (Pin_6), J3.4 (Pin_4)
- net GND: now reaches U.GND
- net GND: now also BZ1.2 (-), J1.1 (Pin_1), J1.2 (Pin_2), J1.7 (Pin_7), J2.1 (Pin_1), J3.3 (Pin_3), R1.2, R2.2
- no-connect marks 0 -> 1
Other:
- moved on the sheet: U

Commit message: PCB design complete
Parts:
- added BATT1: Screw_Terminal_01x02, TerminalBlock_Phoenix:TerminalBlock_Phoenix_MKDS-1,5-2-5.08_1x02_P5.08mm_Horizontal, symbol Connector:Screw_Terminal_01x02
- added C1: 10u, Capacitor_SMD:C_0805_2012Metric_Pad1.18x1.45mm_HandSolder, symbol Device:C
- added C2: 22u, Capacitor_SMD:C_0805_2012Metric_Pad1.18x1.45mm_HandSolder, symbol Device:C
- added U2: AMS1117-5.0, Package_TO_SOT_SMD:SOT-89-3, symbol Regulator_Linear:AMS1117-5.0
- renumbered A to A1, B to B1, U to U1
Connections:
- net +3V3: now also A1.1, B1.1; no longer A1.4, B1.3, B1.4
- net +5V: now also C2.1, U2.2 (VO)
- net BTN_A: now also A1.4; no longer A1.1
- net BTN_B: no longer B1.1
- net GND: now also BATT1.2 (Pin_2), C1.2, C2.2, U2.1 (GND)
- new net VCC: BATT1.1 (Pin_1), C1.1, U2.3 (VI)
